File: hardware/Matrix/Matrix.kicad_sch (KiCad schematic)
At the start: 31 parts, among them J1 IN, J10 Unused 1, J11 Unused 2, J2 OUT, J3 Matrix Out, J4 Power, J5 Power in, J6 Matrix Power, J7 Top LEDs, J8 Bottom LEDs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

Commit message: BG color
Connections:
- net B1: now also J3.1 (Pin_1); no longer J3.5 (Pin_5)
- net B2: now also J3.3 (Pin_3); no longer J3.2 (Pin_2)
- net G1: now also J3.2 (Pin_2); no longer J3.3 (Pin_3)
- net R2: now also J3.5 (Pin_5); no longer J3.1 (Pin_1)
- net P14: now reaches U1.12 (MTMS/GPIO14/ADC2_CH6)
- net P14: now also J1.13 (Pin_13)
- net P12: no longer names the net of U1.13 (MTDI/GPIO12/ADC2_CH5)
- net P12: no longer J1.13 (Pin_13)

Commit message: Almost done with boards
Parts:
- removed J10: Unused 1, Connector_PinSocket_2.54mm:PinSocket_2x03_P2.54mm_Vertical, symbol Connector_Generic:Conn_02x03_Odd_Even
- removed J11: Unused 2, Connector_PinSocket_2.54mm:PinSocket_2x03_P2.54mm_Vertical, symbol Connector_Generic:Conn_02x03_Odd_Even
- removed J3: Matrix Out, Connector_JST:JST_PH_S5B-PH-K_1x05_P2.00mm_Horizontal, symbol Connector_Generic:Conn_01x05
- removed J5: Power in, Custom:JST_VH_B2PS-VH_1x02_P3.96mm_Horizontal, symbol Connector_Generic:Conn_01x02
- removed J6: Matrix Power, Custom:JST_VH_B2PS-VH_1x02_P3.96mm_Horizontal, symbol Connector_Generic:Conn_01x02
- added C1, C2: 100uF, Capacitor_THT:C_Radial_D4.0mm_H5.0mm_P1.50mm, symbol Device:C
- added J10, J11, J12, J13, J14, J15, J16, J17, J18, J6: Conn_01x01, Custom:Single_Pad_2.54mm, symbol Connector_Generic:Conn_01x01
- added J3: Power and Data, Connector_JST:JST_PH_S8B-PH-K_1x08_P2.00mm_Horizontal, symbol Connector_Generic:Conn_01x08
- added J5: Buzzer, Custom:Passive_Buzzer_PCB, symbol Connector_Generic:Conn_01x03
- added R10: 3.9K, Resistor_SMD:R_1206_3216Metric_Pad1.30x1.75mm_HandSolder, symbol Device:R_US
- added R11, R9: 10K, Resistor_SMD:R_1206_3216Metric_Pad1.30x1.75mm_HandSolder, symbol Device:R_US
- added R12: 39K, Resistor_SMD:R_1206_3216Metric_Pad1.30x1.75mm_HandSolder, symbol Device:R_US
- added RV1: 10K, Custom:Potentiometer_Vertical, symbol Device:R_Potentiometer_US
- J7, J8: footprint Connector_JST:JST_PH_S5B-PH-K_1x05_P2.00mm_Horizontal -> Connector_JST:JST_PH_B5B-PH-K_1x05_P2.00mm_Vertical
- J9: footprint Connector_JST:JST_PH_S4B-PH-K_1x04_P2.00mm_Horizontal -> Connector_JST:JST_PH_B4B-PH-K_1x04_P2.00mm_Vertical
Connections:
- net B1: now also J3.4 (Pin_4)
- net B2: now also J3.6 (Pin_6)
- net Earth: now also C1.2, C2.2, J3.1 (Pin_1), J5.1 (Pin_1), R10.2, R12.2, RV1.3
- net G1: now also J3.5 (Pin_5)
- net G2: now also J3.7 (Pin_7)
- net P1: now also J11.1 (Pin_1)
- net P10: now also J14.1 (Pin_1)
- net P17: now also J15.1 (Pin_1)
- net P3: now also J10.1 (Pin_1)
- net P34: now also C1.1, R10.1, R9.2
- net P35: now also C2.1, R11.2, R12.1
- net P36: now also J6.1 (Pin_1)
- net P39: now also J12.1 (Pin_1)
- net P6: now also J18.1 (Pin_1)
- net P7: now also J17.1 (Pin_1)
- net P8: now also J16.1 (Pin_1)
- net P9: now also J13.1 (Pin_1)
- net R2: now also J3.8 (Pin_8)
- net VCC: now also J3.2 (Pin_2), J5.3 (Pin_3)
- net +3V3: now reaches U1.1 (3V3)
- net +3V3: now also RV1.1
- net P12: now reaches U1.13 (MTDI/GPIO12/ADC2_CH5)
- net P12: now also J5.2 (Pin_2)
- new net: R11.1, RV1.2
- new net +BATT: J3.3 (Pin_3), R9.1
Other:
- note added: "Dividing 3.3V to ~2.6V"
- note added: "Dividing 8.4V to ~2.5V"
- moved on the sheet: BT1, BT2, BT3, D1, D2, D3, D4, D5, D6, D7, D8, R1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
