File: hardware/Matrix/Matrix.kicad_pcb (KiCad board)
At the start: 2 copper layers, 66.6 x 88.4 mm, 18 parts, among them J1 IN, J10 Unused 1, J11 Unused 2, J3 Matrix Out, J5 Power in, J6 Matrix Power, J7 Top LEDs, J8 Bottom LEDs, J9 Buttons, U1 ESP32-WROOM

Commit message: BG color
Connections:
- J1 pad 13: /P12 -> /P14
- J3 pad 1: /R2 -> /B1
- J3 pad 2: /B2 -> /G1
- J3 pad 3: /G1 -> /B2
- J3 pad 5: /B1 -> /R2
- U1 pad 12: unconnected-(U1-MTMS/GPIO14/ADC2_CH6-Pad12) -> /P14
- U1 pad 13: /P12 -> unconnected-(U1-MTDI/GPIO12/ADC2_CH5-Pad13)
Routing:
- net /P14: track 0.00 -> 50.2 mm
- net /P12: track 49.1 -> 0.00 mm
- net /B2: track 90.1 -> 80.2 mm
- net /R2: track 79.7 -> 70.4 mm
- net /G2: track 74.0 -> 71.0 mm
- net /G1: track 56.1 -> 54.5 mm
Changed lines of the file:
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@@
 	(net 7 "/B2")
 	(net 8 "/P19")
-	(net 9 "/P12")
+	(net 9 "/P14")
 	(net 10 "/P22")
 	(net 11 "/P18")
@@
 	(net 43 "/P7")
 	(net 44 "/P6")
-	(net 45 "unconnected-(U1-MTMS{slash}GPIO14{slash}ADC2_CH6-Pad12)")
+	(net 45 "unconnected-(U1-MTDI{slash}GPIO12{slash}ADC2_CH5-Pad13)")
 	(net 46 "unconnected-(U1-CHIP_PU-Pad2)")
 	(net 47 "/P8")
@@
 			(layers "*.Cu" "*.Mask")
 			(remove_unused_layers no)
-			(net 45 "unconnected-(U1-MTMS{slash}GPIO14{slash}ADC2_CH6-Pad12)")
+			(net 9 "/P14")
 			(pinfunction "MTMS/GPIO14/ADC2_CH6")
 			(pintype "bidirectional")
@@
 			(layers "*.Cu" "*.Mask")
 			(remove_unused_layers no)
-			(net 9 "/P12")
+			(net 45 "unconnected-(U1-MTDI{slash}GPIO12{slash}ADC2_CH5-Pad13)")
 			(pinfunction "MTDI/GPIO12/ADC2_CH5")
 			(pintype "bidirectional")
@@
 			(remove_unused_layers no)
 			(roundrect_rratio 0.208333)
-			(net 2 "/R2")
+			(net 1 "/B1")
 			(pinfunction "Pin_1")
 			(pintype "passive")
@@
 			(layers "*.Cu" "*.Mask")
 			(remove_unused_layers no)
-			(net 7 "/B2")
+			(net 13 "/G1")
 			(pinfunction "Pin_2")
 			(pintype "passive")
@@
 			(layers "*.Cu" "*.Mask")
 			(remove_unused_layers no)
-			(net 13 "/G1")
+			(net 7 "/B2")
 			(pinfunction "Pin_3")
 			(pintype "passive")
@@
 			(layers "*.Cu" "*.Mask")
 			(remove_unused_layers no)
-			(net 1 "/B1")
+			(net 2 "/R2")
 			(pinfunction "Pin_5")
 			(pintype "passive")
@@
 			(layers "*.Cu" "*.Mask")
 			(remove_unused_layers no)
-			(net 9 "/P12")
+			(net 9 "/P14")
 			(pinfunction "Pin_13")
 			(pintype "passive")
@@
 		)
 	)
-	(gr_text "R2"
+	(gr_text "B1"
 		(at 177.4 63 0)
 		(layer "F.SilkS")
@@
 		)
 	)
-	(gr_text "B1"
+	(gr_text "R2"
 		(at 177.4 55 0)
 		(layer "F.SilkS")
@@
 		)
 	)
-	(gr_text "B2"
+	(gr_text "G1"
 		(at 177.4 61 0)
 		(layer "F.SilkS")
@@
 		)
 	)
-	(gr_text "G1"
+	(gr_text "B2"
 		(at 177.4 59 0)
 		(layer "F.SilkS")
@@
 	)
 	(segment
-		(start 142.484366 65.024)
-		(end 156.708366 50.8)
+		(start 132.08 76.2)
+		(end 133.469 74.811)
 		(width 0.2)
 		(layer "B.Cu")
@@
 	)
 	(segment
-		(start 177.418 50.8)
-		(end 156.708366 50.8)
+		(start 133.469 74.811)
+		(end 133.469 73.18324)
 		(width 0.2)
 		(layer "B.Cu")
@@
 	)
 	(segment
-		(start 133.469 73.18324)
-		(end 141.62824 65.024)
+		(start 182.118 59.436)
+		(end 182.88 60.198)
 		(width 0.2)
 		(layer "B.Cu")
@@
 	)
 	(segment
-		(start 132.08 76.2)
-		(end 133.469 74.811)
+		(start 182.88 60.198)
+		(end 182.88 60.706)
 		(width 0.2)
 		(layer "B.Cu")
@@
 	)
 	(segment
-		(start 133.469 74.811)
-		(end 133.469 73.18324)
+		(start 142.484366 65.024)
+		(end 148.072366 59.436)
 		(width 0.2)
 		(layer "B.Cu")
@@
 	)
 	(segment
-		(start 181.102 54.484)
-		(end 177.418 50.8)
+		(start 148.072366 59.436)
+		(end 182.118 59.436)
 		(width 0.2)
 		(layer "B.Cu")
@@
 	)
 	(segment
-		(start 182.679 53.944694)
-		(end 178.232306 49.498)
+		(start 133.469 73.18324)
+		(end 141.62824 65.024)
 		(width 0.2)
 		(layer "B.Cu")
-		(net 2)
+		(net 1)
 	)
 	(segment
-		(start 182.679 60.907)
-		(end 182.679 53.944694)
+		(start 182.88 60.706)
+		(end 181.102 62.484)
+		(width 0.2)
+		(layer "B.Cu")
+		(net 1)
+	)
+	(segment
+		(start 181.102 52.367694)
+		(end 181.102 54.484)
 		(width 0.2)
 		(layer "B.Cu")
@@
 	)
 	(segment
-		(start 181.102 62.484)
-		(end 182.679 60.907)
+		(start 178.232306 49.498)
+		(end 181.102 52.367694)
 		(width 0.2)
 		(layer "B.Cu")
@@
 	)
 	(segment
-		(start 181.102 60.484)
-		(end 179.926 61.66)
-		(width 0.2)
-		(layer "B.Cu")
-		(net 7)
-	)
-	(segment
-		(start 181.96216 63.385)
-		(end 183.08 62.26716)
-		(width 0.2)
-		(layer "B.Cu")
-		(net 7)
-	)
-	(segment
-		(start 180.24184 63.385)
-		(end 181.96216 63.385)
-		(width 0.2)
-		(layer "B.Cu")
-		(net 7)
-	)
-	(segment
-		(start 179.926 63.06916)
-		(end 180.24184 63.385)
+		(start 180.53 58.484)
+		(end 181.102 58.484)
 		(width 0.2)
 		(layer "B.Cu")
@@
 	)
 	(segment
-		(start 179.926 61.66)
-		(end 179.926 63.06916)
+		(start 178.398406 49.097)
+		(end 182.278 52.976594)
 		(width 0.2)
 		(layer "B.Cu")
@@
 	)
 	(segment
-		(start 130.127 79.327)
-		(end 132.08 81.28)
+		(start 182.278 57.308)
+		(end 181.102 58.484)
 		(width 0.2)
 		(layer "B.Cu")
@@
 	)
 	(segment
-		(start 183.08 62.26716)
-		(end 183.08 53.778594)
+		(start 182.278 52.976594)
+		(end 182.278 57.308)
 		(width 0.2)
 		(layer "B.Cu")
@@
 	)
 	(segment
-		(start 183.08 53.778594)
-		(end 178.398406 49.097)
+		(start 130.127 79.327)
+		(end 132.08 81.28)
 		(width 0.2)
 		(layer "B.Cu")
@@
 	)
 	(segment
-		(start 133.231 86.12124)
-		(end 133.231 87.749)
+		(start 156.579 70.31044)
+		(end 165.1 78.83144)
 		(width 0.2)
 		(layer "B.Cu")
@@
 	)
 	(segment
-		(start 135.09676 85.209)
-		(end 134.14324 85.209)
+		(start 135.771 76.002554)
+		(end 141.463114 70.31044)
 		(width 0.2)
 		(layer "B.Cu")
@@
 	)
 	(segment
-		(start 134.14324 85.209)
+		(start 133.231 87.749)
 		(end 133.231 86.12124)
 		(width 0.2)
@@
 	)
 	(segment
-		(start 133.231 87.749)
-		(end 132.08 88.9)
+		(start 135.09676 85.209)
+		(end 135.771 84.53476)
 		(width 0.2)
 		(layer "B.Cu")
@@
 	)
 	(segment
-		(start 141.463114 70.31044)
-		(end 135.771 76.002554)
+		(start 132.08 88.9)
+		(end 133.231 87.749)
 		(width 0.2)
 		(layer "B.Cu")
@@
 	)
 	(segment
-		(start 135.771 84.53476)
+		(start 134.14324 85.209)
 		(end 135.09676 85.209)
 		(width 0.2)
@@
 	)
 	(segment
-		(start 159.119 70.31044)
-		(end 141.463114 70.31044)
+		(start 141.463114 70.31044)
+		(end 156.579 70.31044)
 		(width 0.2)
 		(layer "B.Cu")
@@
 	)
 	(segment
-		(start 165.1 76.29144)
-		(end 159.119 70.31044)
+		(start 135.771 84.53476)
+		(end 135.771 76.002554)
 		(width 0.2)
 		(layer "B.Cu")
@@
 	)
 	(segment
-		(start 135.771 76.002554)
-		(end 135.771 84.53476)
+		(start 133.231 86.12124)
+		(end 134.14324 85.209)
 		(width 0.2)
 		(layer "B.Cu")
@@
 	)
 	(segment
-		(start 182.278 55.308)
-		(end 182.278 54.110794)
-		(width 0.2)
-		(layer "B.Cu")
-		(net 12)
-	)
-	(segment
-		(start 181.102 56.484)
-		(end 182.278 55.308)
-		(width 0.2)
-		(layer "B.Cu")
-		(net 12)
-	)
-	(segment
 		(start 140.74484 62.69316)
 		(end 130.929 72.509)
@@
 	)
 	(segment
-		(start 178.066206 49.899)
-		(end 155.807366 49.899)
+		(start 174.517 49.899)
+		(end 181.102 56.484)
 		(width 0.2)
 		(layer "B.Cu")
@@
 	)
 	(segment
+		(start 155.807366 49.899)
+		(end 174.517 49.899)
+		(width 0.2)
+		(layer "B.Cu")
+		(net 12)
+	)
+	(segment
 		(start 131.60324 77.351)
 		(end 133.231 77.351)
@@
 	)
 	(segment
-		(start 182.278 54.110794)
-		(end 178.066206 49.899)
-		(width 0.2)
-		(layer "B.Cu")
-		(net 12)
-	)
-	(segment
-		(start 180.53 58.484)
-		(end 181.102 58.484)
-		(width 0.2)
-		(layer "B.Cu")
-		(net 13)
-	)
-	(segment
-		(start 134.62 73.66)
-		(end 138.70756 69.57244)
-		(width 0.2)
-		(layer "B.Cu")
-		(net 13)
-	)
-	(segment
 		(start 138.70756 69.57244)
 		(end 161.786794 69.57244)
@@
 	)
 	(segment
-		(start 167.64 72.644)
-		(end 179.324 60.96)
+		(start 179.8 60.484)
+		(end 181.102 60.484)
 		(width 0.2)
 		(layer "B.Cu")
@@
 	)
 	(segment
-		(start 179.324 60.96)
-		(end 179.324 59.69)
+		(start 167.64 72.644)
+		(end 179.8 60.484)
 		(width 0.2)
 		(layer "B.Cu")
@@
 	)
 	(segment
-		(start 164.858354 72.644)
-		(end 167.64 72.644)
+		(start 134.62 73.66)
+		(end 138.70756 69.57244)
 		(width 0.2)
 		(layer "B.Cu")
@@
 	)
 	(segment
-		(start 179.324 59.69)
-		(end 180.53 58.484)
+		(start 164.858354 72.644)
+		(end 167.64 72.644)
 		(width 0.2)
 		(layer "B.Cu")

Commit message: Almost done with boards
Parts:
- added C1: 100uF, Capacitor_THT:C_Radial_D4.0mm_H5.0mm_P1.50mm, F.Cu at (149.9, 97.8)
- added C2: 100uF, Capacitor_THT:C_Radial_D4.0mm_H5.0mm_P1.50mm, F.Cu at (149.9, 92.7)
- added J12: Conn_01x01, Custom:Single_Pad_2.54mm, F.Cu at (142.2, 99.1)
- added J13: Conn_01x01, Custom:Single_Pad_2.54mm, F.Cu at (142.2, 68.6)
- added J14: Conn_01x01, Custom:Single_Pad_2.54mm, F.Cu at (142.2, 66.0)
- added J15: Conn_01x01, Custom:Single_Pad_2.54mm, F.Cu at (124.5, 81.3)
- added J16: Conn_01x01, Custom:Single_Pad_2.54mm, F.Cu at (124.5, 66.0)
- added J17: Conn_01x01, Custom:Single_Pad_2.54mm, F.Cu at (124.5, 63.5)
- added J18: Conn_01x01, Custom:Single_Pad_2.54mm, F.Cu at (124.5, 61.0)
- added R10: 3.9K, Resistor_SMD:R_1206_3216Metric_Pad1.30x1.75mm_HandSolder, F.Cu at (153.9, 110.7)
- added R11: 10K, Resistor_SMD:R_1206_3216Metric_Pad1.30x1.75mm_HandSolder, F.Cu at (153.7, 79.8)
- added R12: 39K, Resistor_SMD:R_1206_3216Metric_Pad1.30x1.75mm_HandSolder, F.Cu at (153.7, 85.9)
- added R9: 10K, Resistor_SMD:R_1206_3216Metric_Pad1.30x1.75mm_HandSolder, F.Cu at (153.9, 104.9)
- added RV1: 10K, Custom:Potentiometer_Vertical, F.Cu at (160.0, 53.3)
- J10: value Unused 1 -> Conn_01x01; footprint Connector_PinSocket_2.54mm:PinSocket_2x03_P2.54mm_Vertical -> Custom:Single_Pad_2.54mm
- J11: value Unused 2 -> Conn_01x01; footprint Connector_PinSocket_2.54mm:PinSocket_2x03_P2.54mm_Vertical -> Custom:Single_Pad_2.54mm
- J3: value Matrix Out -> Power and Data; footprint Connector_JST:JST_PH_S5B-PH-K_1x05_P2.00mm_Horizontal -> Connector_JST:JST_PH_S8B-PH-K_1x08_P2.00mm_Horizontal
- J5: value Power in -> Buzzer; footprint Custom:JST_VH_B2PS-VH_1x02_P3.96mm_Horizontal -> Custom:Passive_Buzzer_PCB
- J6: value Matrix Power -> Conn_01x01; footprint Custom:JST_VH_B2PS-VH_1x02_P3.96mm_Horizontal -> Custom:Single_Pad_2.54mm
- J7, J8: footprint Connector_JST:JST_PH_S5B-PH-K_1x05_P2.00mm_Horizontal -> Connector_JST:JST_PH_B5B-PH-K_1x05_P2.00mm_Vertical
- J9: footprint Connector_JST:JST_PH_S4B-PH-K_1x04_P2.00mm_Horizontal -> Connector_JST:JST_PH_B4B-PH-K_1x04_P2.00mm_Vertical
- moved J11 46.8 mm to (124.5, 99.1)
- moved J6 36.9 mm to (142.2, 101.6), turned to 0 degrees
- moved J5 25.0 mm to (162.6, 83.8)
- moved R8 23.1 mm to (124.2, 112.5)
- moved R4 23.1 mm to (124.2, 51.8)
- moved R7 21.1 mm to (131.3, 112.5)
- moved R3 21.1 mm to (131.3, 51.8)
- moved J7 20.6 mm to (144.2, 41.1)
- moved U1 20.3 mm to (144.8, 106.7)
- moved R6 19.1 mm to (138.4, 112.5)
- moved R2 19.0 mm to (138.4, 51.8)
- moved J9 17.6 mm to (149.9, 122.7)
- moved J10 17.0 mm to (124.5, 96.5), turned to 0 degrees
- moved R5 16.5 mm to (146.1, 112.5)
- moved R1 16.5 mm to (146.1, 51.8)
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Connections:
- J10 pad 1: /P34 -> /P3
- J11 pad 1: /P6 -> /P1
- J3 pad 1: /B1 -> Earth
- J3 pad 2: /G1 -> VCC
- J3 pad 3: /B2 -> +BATT
- J3 pad 4: /G2 -> /B1
- J3 pad 5: /R2 -> /G1
- J5 pad 2: VCC -> /P12
- J6 pad 1: Earth -> /P36
- U1 pad 1: unconnected-(U1-3V3-Pad1) -> +3V3
- U1 pad 13: unconnected-(U1-MTDI/GPIO12/ADC2_CH5-Pad13) -> /P12
Routing:
- net /P36: track 74.3 -> 2.54 mm
- net /P35: track 85.0 -> 19.5 mm
- net /P10: track 67.7 -> 2.54 mm
- net /P9: track 65.4 -> 2.54 mm
- net +3V3: track 0.00 -> 59.6 mm
- net Earth: track 125.0 -> 183.5 mm
- net /P13: track 70.1 -> 13.8 mm
- net /P39: track 48.0 -> 2.54 mm
- net +BATT: track 0.00 -> 45.2 mm
- net /P17: track 31.6 -> 2.54 mm
- net /B2: track 80.2 -> 51.6 mm
- net Net-(R11-Pad1): track 0.00 -> 24.9 mm
- net /P12: track 0.00 -> 24.2 mm
- net /P34: track 42.7 -> 19.6 mm
- net /P3: track 25.5 -> 2.54 mm
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- added copper zone on In1.Cu, net Earth
- added copper zone on In2.Cu, net Earth
- added copper zone on B.Cu, net VCC
- added copper zone on F.Cu, net VCC
Other:
- board size 66.6 x 88.4 mm -> 56.7 x 88.4 mm
- copper layers 2 -> 4
- board text removed: "B1"
- board text removed: "B2"
- board text removed: "G1"
- board text removed: "G2"
- board text removed: "P1"
- board text removed: "P10"
- board text removed: "P17"
- board text removed: "P3"
- board text removed: "P34"
- board text removed: "P35"
- board text removed: "P36"
- board text removed: "P39"
- board text removed: "P6"
- board text removed: "P7"
- board text removed: "P8"
- board text removed: "P9"
- board text removed: "R2"
- board text removed: "Unused"
- board text removed: "VCC"

Commit message: Maybe done boards?
Parts:
- moved R3 46.2 mm to (155.6, 91.1)
- moved R4 43.0 mm to (148.6, 87.2)
- moved R1 7.97 mm to (138.1, 51.6)
- moved R2 7.35 mm to (131.1, 51.8)
Routing:
- net /LED3: track 12.0 -> 57.1 mm
- net /P33: track 44.1 -> 3.88 mm, vias 2 -> 0
- net /LED4: track 15.8 -> 49.6 mm
- net /P32: track 44.1 -> 11.3 mm, vias 1 -> 0
- net /P2: track 65.6 -> 91.4 mm
- net /P0: track 62.3 -> 84.3 mm
- net /P14: track 41.3 -> 19.4 mm
- net /P4: track 58.9 -> 77.7 mm
- net /P35: track 19.5 -> 36.0 mm
- net /B2: track 51.6 -> 67.9 mm
- net /LED2: track 9.84 -> 25.6 mm
- net /G2: track 49.8 -> 61.3 mm
- net /G1: track 38.3 -> 48.1 mm
- net /LED1: track 10.7 -> 18.3 mm
- net /P27: track 42.9 -> 35.2 mm
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- added copper zone on B.Cu, net Earth
- removed copper zone on In1.Cu, net Earth
- removed copper zone on In2.Cu, net Earth
- removed copper zone on B.Cu, net VCC
- removed copper zone on F.Cu, net VCC
Other:
- copper layers 4 -> 2
